Commit message: Add fence around pursuit area

File: src/dd_robot/urdf/dd_robot.urdf.xacro (robot description, xacro)
@@ -4,5 +4,5 @@
 	<!-- Base Link (Robot Body) -->
 	<link name="base_link">
-		<visual>
+	  <visual>
 			<origin xyz="0 0 0" rpy="0 0 0" />
 			<geometry>
@@ -15,14 +15,42 @@
 		<!-- Collision and Inertia -->
 		<collision>
-      <origin xyz="0 0 0" rpy="0 0 0" />
-      <geometry>
+        <origin xyz="0 0 0" rpy="0 0 0" />
+        <geometry>
           <box size="0.5 0.5 0.25"/>
-      </geometry>
-    </collision>
-    <inertial>
-      <mass value="5"/>
-      <inertia ixx="0.13" ixy="0.0" ixz="0.0" iyy="0.21" iyz="0.0" izz="0.13"/>
-    </inertial>
-	</link>
+        </geometry>
+      </collision>
+      <inertial>
+        <mass value="5"/>
+        <inertia ixx="0.13" ixy="0.0" ixz="0.0" iyy="0.21" iyz="0.0" izz="0.13"/>
+      </inertial>
+	</link>
+	<!-- LiDAR Link -->
+	<link name="laser_frame">
+	  <visual>
+	    <geometry>
+		  <cylinder radius="0.05" length="0.04"/>
+		</geometry>
+		<material name="red">
+		  <color rgba="1 0.2 0.2 1"/>
+		</material>
+	  </visual>
+	  <collision>
+        <geometry>
+		  <cylinder radius="0.05" length="0.04"/>
+		</geometry>
+	  </collision>
+	  <inertial>
+	    <origin xyz="0 0 0" rpy="0 0 0"/>
+		<mass value="0.1"/>
+		<inertia ixx="0.000075" ixy="0.0" ixz="0.0"
+               iyy="0.000075" iyz="0.0"
+               izz="0.000125" />
+	  </inertial>
+	</link>
+	<joint name="laser_joint" type="fixed">
+	  <parent link="base_link"/>
+	  <child link="laser_frame"/>
+	  <origin xyz="0 0 0.225" rpy="0 0 0"/>
+	</joint>
 	<!-- Right Wheel -->
 	<link name="right_wheel">
@@ -83,10 +111,10 @@
 		<axis xyz="0 1 0"/>
 	</joint>
-	<!-- Caster Wheel -->
-	<link name="caster">
+	<!-- Rear Caster Wheel -->
+	<link name="rear_caster">
 		<visual>
 			<origin xyz="0.0 0 0" rpy="0 0 0" />
 			<geometry>
-				<sphere radius="0.05" />
+				<sphere radius="0.07" />
 			</geometry>
 			<material name="darkgray">
@@ -98,5 +126,5 @@
       <origin xyz="0 0 0" rpy="0 0 0" />
       <geometry>
-        <sphere radius="0.05" />
+        <sphere radius="0.07" />
       </geometry>
     </collision>
@@ -106,9 +134,66 @@
     </inertial>
 	</link>
-	<joint name="joint_caster" type="fixed">
-		<parent link="base_link"/>
-		<child link="caster"/>
+	<joint name="joint_front_caster" type="fixed">
+		<parent link="base_link"/>
+		<child link="rear_caster"/>
 		<origin xyz="-0.2 0 -0.125" rpy="0 0 0"/>
 	</joint>
+	<!-- Front Caster Wheel -->
+	<link name="front_caster">
+		<visual>
+			<origin xyz="0.0 0 0" rpy="0 0 0" />
+			<geometry>
+				<sphere radius="0.07" />
+			</geometry>
+			<material name="darkgray">
+				<color rgba="0.2 0.2 0.2 1"/>
+			</material>
+		</visual>
+		<!-- Collision and Inertia -->
+		<collision>
+      <origin xyz="0 0 0" rpy="0 0 0" />
+      <geometry>
+        <sphere radius="0.07" />
+      </geometry>
+    </collision>
+    <inertial>
+      <mass value="0.5"/>
+      <inertia ixx="0.0001" ixy="0.0" ixz="0.0" iyy="0.0001" iyz="0.0" izz="0.0001"/>
+    </inertial>
+	</link>
+	<joint name="joint_rear_caster" type="fixed">
+		<parent link="base_link"/>
+		<child link="front_caster"/>
+		<origin xyz="0.2 0 -0.125" rpy="0 0 0"/>
+	</joint>
+	<!-- LiDAR Sensor Definition -->
+	<gazebo reference="laser_frame">
+	  <sensor name="lidar" type="lidar">
+	    <topic>/model/$(arg robot_name)/scan</topic>
+		<update_rate>10</update_rate>
+		<lidar>
+		  <scan>
+		    <horizontal>
+			  <samples>360</samples>
+			  <resolution>1</resolution>
+			  <min_angle>-3.14159</min_angle>
+			  <max_angle>3.14159</max_angle>
+			</horizontal>
+		  </scan>
+		  <range>
+		    <min>0.15</min>
+			<max>12.0</max>
+			<resolution>0.01</resolution>
+		  </range>
+		  <noise>
+		    <type>gaussian</type>
+			<mean>0.0</mean>
+			<stddev>0.01</stddev>
+		  </noise>
+		</lidar>
+		<always_on>1</always_on>
+		<visualize>true</visualize>
+	  </sensor>
+	</gazebo>
 	<!-- Communicating with Gazebo -->
 	<gazebo>
@@ -138,8 +223,15 @@
       		<update_frequency>10</update_frequency>
     	</plugin>
-	</gazebo>
-	<gazebo reference="caster">
+		<plugin filename="gz-sim-sensors-system" name="gz::sim::systems::Sensors">
+		    <render_engine>ogre1</render_engine>
+		</plugin>
+	</gazebo>
+	<gazebo reference="rear_caster">
 		<mul1>0.0</mul1>
 		<mul2>0.0</mul2>
 	</gazebo>
+	<gazebo reference="front_caster">
+		<mul1>0.0</mul1>
+		<mul2>0.0</mul2>
+	</gazebo>
 </robot>

Commit message: all workcode

File: src/dd_robot/urdf/dd_robot.urdf.xacro (robot description, xacro)
@@ -9,7 +9,14 @@
 				<box size="0.5 0.5 0.25" />
 			</geometry>
-			<material name="blue">
-				<color rgba="0 0.5 1 1"/>
-			</material>
+			<xacro:if value="${'$(arg robot_name)'.startswith('evader')}">
+				<material name="red">
+					<color rgba="1 0 0 1"/>
+				</material>
+			</xacro:if>
+			<xacro:unless value="${'$(arg robot_name)'.startswith('evader')}">
+				<material name="blue">
+					<color rgba="0 0.5 1 1"/>
+				</material>
+			</xacro:unless>
 		</visual>
 		<!-- Collision and Inertia -->
@@ -36,7 +43,9 @@
 	  </visual>
 	  <collision>
-        <geometry>
-		  <cylinder radius="0.05" length="0.04"/>
-		</geometry>
+		<xacro:if value="${'$(arg robot_name)'.startswith('pursuer')}">
+			<geometry>
+				<cylinder radius="0.05" length="0.04"/>
+			</geometry>
+		</xacro:if>
 	  </collision>
 	  <inertial>
